Commit message: added 2 passive caster wheels

File: robots/tractor.urdf.xacro (robot description, xacro)
@@ -10,5 +10,5 @@
  <xacro:include filename="$(find tractor_description)/robots/maxii.xacro"/>
   <xacro:include filename="$(find tractor_description)/urdfs/front_wheel.xacro"/>
-  <xacro:include filename="$(find tractor_description)/urdfs/rear_wheel.xacro"/>
+  <xacro:include filename="$(find tractor_description)/urdfs/caster_wheel.xacro"/>
   <!-- Accessories -->
   <xacro:include filename="$(find tractor_description)/urdfs/accessories/gps.xacro"/>
@@ -20,8 +20,8 @@
   <xacro:property name="position_right" value="-0.315" />
   <xacro:maxii/>
-  <xacro:front_wheel left_right="left" radius="0.15" length="0.13" position="${position_left}"/>
-  <xacro:front_wheel left_right="right" radius="0.15" length="0.13" position="${position_right}"/>
-  <xacro:rear_wheel left_right="left" radius="0.12" length="0.13" position="${position_left}"/>
-  <xacro:rear_wheel left_right="right" radius="0.12" length="0.13" position="${position_right}"/>
+  <xacro:front_wheel left_right="left" radius="0.0856" length="0.13" position="${position_left}"/>
+  <xacro:front_wheel left_right="right" radius="0.0856" length="0.13" position="${position_right}"/>
+  <xacro:caster_wheel name="front" translateX="0.2" translateY="0." radius="0.025" length="0.02"/>
+  <xacro:caster_wheel name="back" translateX="-0.3" translateY="0." radius="0.025" length="0.02"/>
   <!-- SENSORS-->
   <!--xacro:robot_gps x="0.05" y="0" z="0.1875" gps_size="0.1"/-->

File: urdfs/caster_wheel.xacro (robot description, xacro)
@@ -2,7 +2,7 @@
 <robot xmlns:xacro="http://www.ros.org/wiki/xacro" name="front_wheel">
 <xacro:include filename="$(find tractor_description)/urdfs/cylinder_inertia.xacro"/>
-<xacro:macro name="front_wheel" params="left_right radius length position">
-    <xacro:property name="mass" value="4" />
-    <link name="front_${left_right}_wheel">
+<xacro:macro name="caster_wheel" params="name translateX translateY radius length">
+    <xacro:property name="mass" value="0.5" />
+    <link name="${name}_caster_wheel">
        <visual>
             <geometry>
@@ -17,22 +17,12 @@
         <xacro:cylinder_inertia mass="${mass}" radius="${radius}" length="${length}"/>
     </link>
-    <joint name="front_${left_right}_wheel_joint" type="continuous">
-        <origin xyz="0.0 ${position} -0.17" rpy=" -1.57 0 0" />
+    <joint name="${name}_caster_wheel_joint" type="continuous">
+        <origin xyz="${translateX}  ${translateY} -0.23" rpy=" -1.57 0 0" />
         <parent link="base_link" />
-        <child link="front_${left_right}_wheel" />
+        <child link="${name}_caster_wheel" />
         <axis  xyz="0 0 1" />
 	<dynamics damping="0" friction="0"/>
     </joint>
-    <transmission name="trans_front_${left_right}_wheel">
-        <type>transmission_interface/SimpleTransmission</type>
-        <joint name="front_${left_right}_wheel_joint">
-        <!--hardwareInterface>hardware_interface/VelocityJointInterface</hardwareInterface-->
-	<hardwareInterface>hardware_interface/EffortJointInterface</hardwareInterface>
-        </joint>
-        <actuator name="motor_front_${left_right}_wheel">
-        <mechanicalReduction>1</mechanicalReduction>
-        </actuator>
-    </transmission>
-    <gazebo reference="front_${left_right}_wheel">
+    <gazebo reference="${name}_caster_wheel">
         <gravity>true</gravity>
         <mu1>1</mu1>

Commit message: added velodyne to robot using wolf version

File: robots/tractor.urdf.xacro (robot description, xacro)
@@ -1,7 +1,6 @@
 <?xml version="1.0" ?>
 <robot name="tractor" xmlns:xacro="http://ros.org/wiki/xacro">
-    <!--- new_gazebo_version should be false by default because pinocchio needs it!-->
     <xacro:arg name="robot_name" default="tractor"/>
-    <xacro:arg name="new_gazebo_version" default="false"/>
+    <xacro:arg name="sensors" default="true"/>
     <xacro:include filename="$(find myrobot_description)/gazebo/gazebo.urdf.xacro">
         <xacro:arg name="task_period" value="$(arg task_period)"/>
@@ -18,8 +17,8 @@
   <xacro:include filename="$(find tractor_description)/urdfs/accessories/velodyne_vlp16.xacro"/>
   <xacro:property name="position_left" value="0.305" />
-  <xacro:property name="position_right" value="-0.315" />
+  <xacro:property name="position_right" value="-0.305" />
   <xacro:maxii/>
-  <xacro:front_wheel left_right="left" radius="0.0856" length="0.13" position="${position_left}"/>
-  <xacro:front_wheel left_right="right" radius="0.0856" length="0.13" position="${position_right}"/>
+  <xacro:front_wheel left_right="left" radius="0.0856" length="0.02" position="${position_left}"/>
+  <xacro:front_wheel left_right="right" radius="0.0856" length="0.02" position="${position_right}"/>
   <xacro:caster_wheel name="front" translateX="0.2" translateY="0." radius="0.025" length="0.02"/>
   <xacro:caster_wheel name="back" translateX="-0.3" translateY="0." radius="0.025" length="0.02"/>
@@ -29,4 +28,9 @@
   <!-- <xacro:robot_laser x="0.0" y="0.0" z="0.245" laser_size="0.1"/> -->
   <!--xacro:intel_realsense x="0.1" y="0.0" z="0.5"/-->
-  <!--xacro:velodyne_vlp16/-->
+     <xacro:if value="$(arg sensors)">
+          <xacro:VLP-16 parent="base_link" name="rslidar" topic="/$(arg robot_name)/lidar_points"
+                organize_cloud="true" hz="10" gpu="true">
+    	  <origin xyz="0.0 0 0.1" rpy="0 0 0" />
+  	</xacro:VLP-16>
+    </xacro:if>
 </robot>

File: urdfs/accessories/velodyne_vlp16.xacro (robot description, xacro)
@@ -1,7 +1,12 @@
 <?xml version="1.0"?>
-<robot xmlns:xacro="http://www.ros.org/wiki/xacro" name="robot_laser">
+<robot xmlns:xacro="http://www.ros.org/wiki/xacro" name="VLP-16">
   <xacro:property name="M_PI" value="3.1415926535897931" />
-  <xacro:macro name="velodyne_vlp16">
-    <link name="velodyne_vlp16_base_link">
+  <xacro:macro name="VLP-16" params="*origin parent:=base_link name:=velodyne topic:=/velodyne_points organize_cloud:=false hz:=10 lasers:=16 samples:=1875 collision_range:=0.3 min_range:=0.9 max_range:=130.0 noise:=0.008 min_angle:=-${M_PI} max_angle:=${M_PI} gpu:=false">
+    <joint name="${name}_base_mount_joint" type="fixed">
+      <xacro:insert_block name="origin" />
+      <parent link="${parent}"/>
+      <child link="${name}_base_link"/>
+    </joint>
+    <link name="${name}_base_link">
       <inertial>
         <mass value="0.83"/>
@@ -28,10 +33,10 @@
       </collision>
     </link>
-    <joint name="velodyne_vlp16_base_joint" type="fixed" >
-      <origin xyz="-0.03 0 0.2" rpy="0 0 0" />
-      <parent link="base_link" />
-      <child link="velodyne_vlp16_base_link"/>
+    <joint name="${name}_base_scan_joint" type="fixed" >
+      <origin xyz="0 0 0.0377" rpy="0 0 0" />
+      <parent link="${name}_base_link" />
+      <child link="${name}"/>
     </joint>
-    <link name="velodyne_vlp16">
+    <link name="${name}">
       <inertial>
         <mass value="0.01"/>
@@ -45,25 +50,27 @@
         </geometry>
       </visual>
+      <collision>
+        <geometry>
+          <sphere radius="0"/>
+        </geometry>
+      </collision>
     </link>
-    <joint name="velodyne_vlp16_joint" type="fixed" >
-      <origin xyz="0 0 0.0377" rpy="0 0 0" />
-      <parent link="velodyne_vlp16_base_link" />
-      <child link="velodyne_vlp16"/>
-    </joint>
-    <gazebo reference="velodyne_vlp16">
-        <sensor type="gpu_ray" name="VLP16">
+    <!-- Gazebo requires the velodyne_gazebo_plugins package -->
+    <gazebo reference="${name}">
+      <xacro:if value="${gpu}">
+        <sensor type="gpu_ray" name="${name}-VLP16">
           <pose>0 0 0 0 0 0</pose>
           <visualize>false</visualize>
-          <update_rate>10</update_rate>
+          <update_rate>${hz}</update_rate>
           <ray>
             <scan>
               <horizontal>
-                <samples>360</samples>
+                <samples>${samples}</samples>
                 <resolution>1</resolution>
-                <min_angle>${-M_PI}</min_angle>
-                <max_angle>${M_PI}</max_angle>
+                <min_angle>${min_angle}</min_angle>
+                <max_angle>${max_angle}</max_angle>
               </horizontal>
               <vertical>
-                <samples>16</samples>
+                <samples>${lasers}</samples>
                 <resolution>1</resolution>
                 <min_angle>-${15.0*M_PI/180.0}</min_angle>
@@ -72,6 +79,6 @@
             </scan>
             <range>
-              <min>1</min>
-              <max>140</max>
+              <min>${collision_range}</min>
+              <max>${max_range+1}</max>
               <resolution>0.001</resolution>
             </range>
@@ -83,11 +90,54 @@
           </ray>
           <plugin name="gazebo_ros_laser_controller" filename="libgazebo_ros_velodyne_gpu_laser.so">
-            <topicName>robot/velodyne</topicName>
-            <frameName>velodyne_vlp16</frameName>
-            <min_range>1</min_range>
-            <max_range>140</max_range>
-            <gaussianNoise>0.008</gaussianNoise>
+            <topicName>${topic}</topicName>
+            <frameName>${name}</frameName>
+            <organize_cloud>${organize_cloud}</organize_cloud>
+            <min_range>${min_range}</min_range>
+            <max_range>${max_range}</max_range>
+            <gaussianNoise>${noise}</gaussianNoise>
           </plugin>
         </sensor>
+      </xacro:if>
+      <xacro:unless value="${gpu}">
+        <sensor type="ray" name="${name}-VLP16">
+          <pose>0 0 0 0 0 0</pose>
+          <visualize>false</visualize>
+          <update_rate>${hz}</update_rate>
+          <ray>
+            <scan>
+              <horizontal>
+                <samples>${samples}</samples>
+                <resolution>1</resolution>
+                <min_angle>${min_angle}</min_angle>
+                <max_angle>${max_angle}</max_angle>
+              </horizontal>
+              <vertical>
+                <samples>${lasers}</samples>
+                <resolution>1</resolution>
+                <min_angle>-${15.0*M_PI/180.0}</min_angle>
+                <max_angle> ${15.0*M_PI/180.0}</max_angle>
+              </vertical>
+            </scan>
+            <range>
+              <min>${collision_range}</min>
+              <max>${max_range+1}</max>
+              <resolution>0.001</resolution>
+            </range>
+            <noise>
+              <type>gaussian</type>
+              <mean>0.0</mean>
+              <stddev>0.0</stddev>
+            </noise>
+          </ray>
+          <plugin name="gazebo_ros_laser_controller" filename="libgazebo_ros_velodyne_laser.so">
+            <topicName>${topic}</topicName>
+            <frameName>${name}</frameName>
+            <organize_cloud>${organize_cloud}</organize_cloud>
+            <min_range>${min_range}</min_range>
+            <max_range>${max_range}</max_range>
+            <gaussianNoise>${noise}</gaussianNoise>
+          </plugin>
+        </sensor>
+      </xacro:unless>
     </gazebo>
   </xacro:macro>

Commit message: elevated velodyne
differentiating friction models

File: robots/tractor.urdf.xacro (robot description, xacro)
@@ -31,5 +31,5 @@
           <xacro:VLP-16 parent="base_link" name="rslidar" topic="/$(arg robot_name)/lidar_points"
                 organize_cloud="true" hz="10" gpu="true">
-    	  <origin xyz="0.0 0 0.1" rpy="0 0 0" />
+    	  <origin xyz="0.0 0 0.3" rpy="0 0 0" />
   	</xacro:VLP-16>
     </xacro:if>

Commit message: added possibility to have arm on top

File: robots/tractor.urdf.xacro (robot description, xacro)
@@ -1,6 +1,7 @@
 <?xml version="1.0" ?>
 <robot name="tractor" xmlns:xacro="http://ros.org/wiki/xacro">
-    <xacro:arg name="robot_name" default="tractor"/>
-    <xacro:arg name="sensors" default="true"/>
+	<xacro:arg name="robot_name" default="tractor"/>
+	<xacro:arg name="sensors" default="true"/>
+	<xacro:arg name="arm" default="false"/>
     <xacro:include filename="$(find myrobot_description)/gazebo/gazebo.urdf.xacro">
         <xacro:arg name="task_period" value="$(arg task_period)"/>
@@ -23,4 +24,10 @@
   <xacro:caster_wheel name="front" translateX="0.2" translateY="0." radius="0.025" length="0.02"/>
   <xacro:caster_wheel name="back" translateX="-0.3" translateY="0." radius="0.025" length="0.02"/>
+  <xacro:if value="$(arg arm)">
+   	<xacro:include filename="$(find z1_description)/xacro/z1_arm.xacro"/>
+	<xacro:z1_arm parent="base_link">
+		<origin xyz="0 0 0.15" rpy="0 0 0"/>
+	</xacro:z1_arm>
+ </xacro:if>
   <!-- SENSORS-->
   <!--xacro:robot_gps x="0.05" y="0" z="0.1875" gps_size="0.1"/-->
