Commit message: transmission is now 1
added visual for wheels

File: robots/maxii.xacro (robot description, xacro)
@@ -392,9 +392,9 @@
     </joint>
     <link name="ruota_motrice2">
-      <!-- <inertial>
+      <inertial>
         <origin xyz="0.26377726016691 0.128486306304607 -0.043300885340771" rpy="0 0 0" />
         <mass value="0.352270876846932" />
         <inertia ixx="0.000552782855065526" ixy="-1.57290978416372E-18" ixz="3.14137307635142E-21" iyy="0.000552782855065525" iyz="-1.8574920937579E-21" izz="0.00108208098500792" />
-      </inertial> -->
+      </inertial>
       <visual>
         <origin xyz="0 0 0"  rpy="0 0 0" />

File: urdfs/front_wheel.xacro (robot description, xacro)
@@ -5,9 +5,9 @@
     <xacro:property name="mass" value="4" />
     <link name="front_${left_right}_wheel">
-        <!-- <visual>
+       <visual>
             <geometry>
                 <cylinder radius="${radius}" length="${length}" />
             </geometry>
-        </visual> -->
+        </visual>
         <collision>
             <geometry>
@@ -30,5 +30,5 @@
         </joint>
         <actuator name="motor_front_${left_right}_wheel">
-        <mechanicalReduction>100</mechanicalReduction>
+        <mechanicalReduction>1</mechanicalReduction>
         </actuator>
     </transmission>

File: urdfs/rear_wheel.xacro (robot description, xacro)
@@ -5,9 +5,9 @@
     <xacro:property name="mass" value="4.23900913" />
     <link name="rear_${left_right}_wheel">
-        <!-- <visual>
+        <visual>
             <geometry>
                 <cylinder radius="${radius}" length="${length}" />
             </geometry>
-        </visual> -->
+        </visual>
         <collision>
             <geometry>
@@ -30,5 +30,5 @@
         </joint>
         <actuator name="motor_rear_${left_right}_wheel">
-        <mechanicalReduction>100</mechanicalReduction>
+        <mechanicalReduction>1</mechanicalReduction>
         </actuator>
     </transmission>

Commit message: added coppeliasim models

File: robots/maxii.xacro (robot description, xacro)
@@ -84,10 +84,10 @@
         <material name="grey"/>
       </visual>
-      <collision>
+      <!--collision>
         <origin xyz="0 0 0" rpy="0 0 0" />
         <geometry>
           <mesh filename="package://tractor_description/meshes/meshes1/cingolo1.STL" />
         </geometry>
-      </collision>
+      </collision-->
     </link>
     <joint name="cingolo1_joint" type="fixed">
@@ -269,10 +269,10 @@
         <material name="grey"/>
       </visual>
-      <collision>
+      <!--collision>
         <origin xyz="0 0 0" rpy="0 0 0" />
         <geometry>
           <mesh filename="package://tractor_description/meshes/meshes2/cingolo2.STL" />
         </geometry>
-      </collision>
+      </collision-->
     </link>
     <joint name="cingolo2_joint"  type="fixed">

Commit message: aligned baseframe to medium point of tracks

File: robots/maxii.xacro (robot description, xacro)
@@ -17,4 +17,5 @@
       <color rgba="0 0 0 1.0"/>
     </material>
+   <xacro:arg name="base_offset" default="0.08"/>
     <link name = "base_link">
     </link>
@@ -40,5 +41,5 @@
     </link>
     <joint name="chassis_joint" type="fixed">
-      <origin xyz="0 0.225 0" rpy="0 0 0" />
+      <origin xyz="$(arg base_offset) 0.225 0" rpy="0 0 0" />
       <parent link="base_link" />
       <child link="chassis" />
@@ -66,5 +67,5 @@
     </link>
     <joint name="ponte1_joint" type="fixed">
-      <origin xyz="0 0.225 0" rpy="0 0 0" />
+      <origin xyz="$(arg base_offset) 0.225 0" rpy="0 0 0" />
       <parent link="base_link" />
       <child link="ponte1" />
@@ -92,5 +93,5 @@
     </link>
     <joint name="cingolo1_joint" type="fixed">
-      <origin xyz="-0.094340414586262 -0.301388567 -0.100112309063136" rpy="1.5707963267949 0 3.14" />
+      <origin xyz="${$(arg base_offset) -0.094340414586262} -0.301388567 -0.100112309063136" rpy="1.5707963267949 0 3.14" />
       <parent link="base_link" />
       <child link="cingolo1" />
@@ -118,5 +119,5 @@
     </link>
     <joint name="supporto_ruote1_joint" type="fixed">
-      <origin xyz="-0.249653977391183 -0.353238567 -0.0779139783362333" rpy="-2.45232668596043 0 1.57" />
+      <origin xyz="${$(arg base_offset)-0.249653977391183} -0.353238567 -0.0779139783362333" rpy="-2.45232668596043 0 1.57" />
       <parent link="base_link" />
       <child link="supporto_ruote1" />
@@ -148,5 +149,5 @@
     </link>
     <joint name="sospensioni1_joint" type="fixed">
-      <origin xyz="0.115815637360445 -0.300738567 -0.0224356268106508" rpy="-1.91368272087089 0 -1.5707963267949" />
+      <origin xyz="${$(arg base_offset) + 0.115815637360445} -0.300738567 -0.0224356268106508" rpy="-1.91368272087089 0 -1.5707963267949" />
       <parent link="base_link" />
       <child link="sospensioni1" />
@@ -174,5 +175,5 @@
     </link>
     <joint name="assi1_joint" type="fixed">
-      <origin xyz="-0.399632572527583 -0.302738567 -0.131814051628503" rpy="-1.91580745395575 0 1.57" />
+      <origin xyz="${$(arg base_offset) -0.399632572527583} -0.302738567 -0.131814051628503" rpy="-1.91580745395575 0 1.57" />
       <parent link="base_link" />
       <child link="assi1" />
@@ -200,5 +201,5 @@
     </link>
     <joint name="ruote_folli1_joint" type="fixed">
-      <origin xyz="-0.399632572527583 -0.302738567 -0.131814051628503" rpy="-1.5707963267949 -1.29575751456647 3.14" />
+      <origin xyz="${$(arg base_offset)-0.399632572527583} -0.302738567 -0.131814051628503" rpy="-1.5707963267949 -1.29575751456647 3.14" />
       <parent link="base_link" />
       <child link="ruote_folli1" />
@@ -226,5 +227,5 @@
     </link>
     <joint name="ruota_motrice1_joint" type="fixed">
-      <origin xyz="-0.096734450942382 -0.286388567 0.087326977068925" rpy="-1.5707963267949 -1.22950532384837 3.14" />
+      <origin xyz="${$(arg base_offset)-0.096734450942382} -0.286388567 0.087326977068925" rpy="-1.5707963267949 -1.22950532384837 3.14" />
       <parent link="base_link" />
       <child link="ruota_motrice1" />
@@ -251,5 +252,5 @@
     </link>
     <joint name="ponte2_joint" type="fixed">
-      <origin xyz="0 0.225 0" rpy="0 0 0" />
+      <origin xyz="$(arg base_offset) 0.225 0" rpy="0 0 0" />
       <parent link="base_link" />
       <child link="ponte2" />
@@ -258,5 +259,5 @@
     <link name="cingolo2">
       <inertial>
-        <origin xyz="-0.0186478543961228 0.0173558435086227 -8.32667268468867E-17" rpy="0 0 0" />
+        <origin xyz="${$(arg base_offset)-0.0186478543961228} 0.0173558435086227 -8.32667268468867E-17" rpy="0 0 0" />
         <mass value="5.37116770201881" />
         <inertia ixx="0.119835058050815" ixy="0.0195379499468073" ixz="8.99361040190704E-17" iyy="0.414599681845954" iyz="3.60868166771734E-17" izz="0.519305950869416" />
@@ -277,5 +278,5 @@
     </link>
     <joint name="cingolo2_joint"  type="fixed">
-      <origin xyz="-0.094340414586137 0.31585 -0.100112309063133" rpy="1.57079632679489 0 3.14" />
+      <origin xyz="${$(arg base_offset)-0.094340414586137} 0.31585 -0.100112309063133" rpy="1.57079632679489 0 3.14" />
       <parent link="base_link" />
       <child link="cingolo2" />
@@ -307,5 +308,5 @@
     </link>
     <joint name="sospensioni2_joint"  type="fixed">
-      <origin  xyz="0.115815637360568 0.3165 -0.022435626810643" rpy="-1.91368272087087 0 -1.5707963267949" />
+      <origin  xyz="${$(arg base_offset)+0.115815637360568} 0.3165 -0.022435626810643" rpy="-1.91368272087087 0 -1.5707963267949" />
       <parent link="base_link" />
       <child link="sospensioni2" />
@@ -333,5 +334,5 @@
     </link>
     <joint name="supporto_ruote2_joint" type="fixed">
-      <origin xyz="-0.249653977391059 0.264 -0.0779139783362343" rpy="-2.45232668596046 0 1.57" />
+      <origin xyz="${$(arg base_offset)-0.249653977391059} 0.264 -0.0779139783362343" rpy="-2.45232668596046 0 1.57" />
       <parent link="base_link" />
       <child link="supporto_ruote2" />
@@ -360,5 +361,5 @@
     </link>
     <joint  name="assi2_joint" type="fixed">
-      <origin xyz="-0.249653977391059 0.3145 -0.077913978336234" rpy="3.06127497605204 0 1.57" />
+      <origin xyz="${$(arg base_offset)-0.249653977391059} 0.3145 -0.077913978336234" rpy="3.06127497605204 0 1.57" />
       <parent link="base_link" />
       <child link="assi2" />
@@ -386,5 +387,5 @@
     </link>
     <joint name="ruote_folli2_joint" type="fixed">
-      <origin xyz="-0.382705304353283 0.2915 -0.127037337056396" rpy="-1.5707963267949 -1.29575751456645 3.14" />
+      <origin xyz="${$(arg base_offset)-0.382705304353283} 0.2915 -0.127037337056396" rpy="-1.5707963267949 -1.29575751456645 3.14" />
       <parent link="base_link" />
       <child link="ruote_folli2" />
@@ -412,5 +413,5 @@
     </link>
     <joint name="ruota_motrice2_joint" type="fixed">
-      <origin  xyz="-0.360511711109277 0.275382964 -0.041159329235658" rpy="1.5707963267949 0 0" />
+      <origin  xyz="${$(arg base_offset)-0.360511711109277} 0.275382964 -0.041159329235658" rpy="1.5707963267949 0 0" />
       <parent link="base_link" />
       <child link="ruota_motrice2" />
