Commit message: commented visual for caster wheel that was a ugly white cylinder in WF
added ramp irdf
updated rviz config for paper

File: urdfs/caster_wheel.xacro (robot description, xacro)
@@ -5,9 +5,4 @@
     <xacro:property name="mass" value="0.5" />
     <link name="${name}_caster_wheel">
-       <visual>
-            <geometry>
-                <cylinder radius="${radius}" length="${length}" />
-            </geometry>
-        </visual>
         <collision>
             <geometry>

File: urdfs/front_wheel.xacro (robot description, xacro)
@@ -5,9 +5,4 @@
     <xacro:property name="mass" value="4" />
     <link name="front_${left_right}_wheel">
-       <visual>
-            <geometry>
-                <cylinder radius="${radius}" length="${length}" />
-            </geometry>
-        </visual>
         <collision>
             <geometry>
